File: Designs/MAX86141HEG/MAX86141_HEG_MINI.brd (EAGLE design)
At the start: 65 x 9.9 mm, 18 parts, among them U1 MAX86141ENP+T, U3 TXBN0304RUTR, U4 LP5907MFX-3.3/NOPB

Commit message: fixes in design I'm testing
Parts:
- moved JP2 5.00 mm to (127.8, 20.1)
- moved JP3 5.00 mm to (127.8, 13.6)
Routing:
- net GND: track 74.5 -> 108.6 mm, vias 2 -> 3
- net INT: track 27.9 -> 50.0 mm, vias 1 -> 2
- net SDO3.3: track 15.9 -> 37.4 mm, vias 1 -> 2
- net 3.3V: track 70.5 -> 91.1 mm, vias 3 -> 4
- net CSB3.3: track 21.2 -> 40.9 mm, vias 1 -> 2
- net SCLK3.3: track 12.8 -> 31.3 mm, vias 1 -> 2
- net SDI3.3: track 18.9 -> 36.7 mm, vias 1 -> 2
- net GPIO1: track 25.5 -> 42.9 mm, vias 1 -> 2
- net GPIO2: track 22.7 -> 39.8 mm, vias 1 -> 2
- net PD_GND: track 29.1 -> 42.8 mm, vias 2 -> 3
Other:
- board size 65 x 9.9 mm -> 70 x 9.9 mm

Commit message: Update MAX86141_HEG_MINI.brd
Changed lines of the file:
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@@
 <setting verticaltext="up"/>
 </settings>
-<grid distance="20" unitdist="mil" unit="mil" style="lines" multiple="1" display="no" altdistance="5" altunitdist="mil" altunit="mil"/>
+<grid distance="1" unitdist="mil" unit="mil" style="lines" multiple="1" display="no" altdistance="5" altunitdist="mil" altunit="mil"/>
 <layers>
 <layer number="1" name="Top" color="4" fill="1" visible="yes" active="yes"/>
@@
 <wire x1="124.587" y1="20.4216" x2="124.6632" y2="20.4978" width="0.508" layer="16"/>
 <wire x1="124.6632" y1="20.4978" x2="124.7902" y2="20.4978" width="0.508" layer="16"/>
-<wire x1="126.365" y1="19.0246" x2="126.365" y2="20.2946" width="0.508" layer="1"/>
-<wire x1="126.5682" y1="20.4978" x2="126.365" y2="20.2946" width="0.508" layer="1"/>
-<wire x1="127.8128" y1="18.9992" x2="127.2921" y2="18.4785" width="0.508" layer="1"/>
-<wire x1="127.8128" y1="18.9992" x2="127.8128" y2="20.4978" width="0.508" layer="1"/>
-<wire x1="127.8128" y1="20.4978" x2="126.5682" y2="20.4978" width="0.508" layer="1"/>
-<wire x1="125.2474" y1="19.4056" x2="126.365" y2="19.0246" width="0" layer="19" extent="1-16"/>
+<wire x1="125.2474" y1="18.3642" x2="124.714" y2="18.8976" width="0.8128" layer="1"/>
+<wire x1="124.714" y1="18.8976" x2="124.714" y2="20.3708" width="0.8128" layer="1"/>
+<wire x1="125.5141" y1="18.0975" x2="125.5141" y2="18.3261" width="0.8128" layer="1"/>
+<wire x1="125.5141" y1="18.3261" x2="125.8824" y2="18.6944" width="0.8128" layer="1"/>
+<wire x1="125.8824" y1="18.6944" x2="125.8824" y2="20.3962" width="0.8128" layer="1"/>
 </signal>
 <signal name="GPIO2">

Commit message: updates/another fix for boot routine
Parts:
- removed LED1, LED2: (no value), led:CHIPLED_1206
- added L1, L2, L3: (no value), led:CHIPLED_1206
Connections:
- new net LED1: L1.C, U1.D1
- net 3.3V: now also L1.A, L2.A, L3.A; no longer LED1.A, LED2.A
- net LED2: now also L2.C; no longer LED1.C
- net LED3: now also L3.C; no longer LED2.C
Routing:
- net LED1: track 0.00 -> 37.5 mm
- net 3.3V: track 91.1 -> 95.2 mm
Other:
- board size 70 x 9.9 mm -> 76 x 10 mm
- board text added: "L1 L2 L3"

Commit message: quality improvements to design (hopefully)
Parts:
- U1: device MAX86141:21-100134A_20 -> MAX86141:21-100134_N201A2-1_MXM
Routing:
- net GPIO2: track 39.8 -> 41.8 mm
- net INT: track 50.0 -> 51.0 mm
- net 3.3V: track 95.2 -> 94.5 mm

Commit message: reverted breakout board (trace spacing too narrow)
Parts:
- U1: device MAX86141:21-100134_N201A2-1_MXM -> MAX86141:21-100134A_20
Routing:
- net GPIO2: track 41.8 -> 39.8 mm
- net INT: track 51.0 -> 50.0 mm
- net 3.3V: track 94.5 -> 95.2 mm
